File: HARDWARE/ServoDriver/ArmDriver.kicad_pcb (KiCad board)
At the start: 2 copper layers, 106.6 x 66 mm, 48 parts, among them J1 Conn_01x03_Male, J10 Screw_Terminal_01x02, J2 Conn_01x03_Male, J3 Conn_01x03_Male, J4 Conn_01x03_Male, J5 Conn_01x03_Male, J6 Conn_01x03_Male, J7 Conn_01x03_Male, J8 Conn_01x03_Male, J9 I2C Connector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

Commit message: ArmDriver rev2
Parts:
- removed REF** (x4): MountingHole_2.2mm_M2, MountingHole:MountingHole_2.2mm_M2
- added J11: Fan Connector, Connector_PinHeader_2.54mm:PinHeader_1x02_P2.54mm_Vertical, F.Cu at (175.3, 81.3)
- added REF0: MountingHole_2.2mm_M2, MountingHole:MountingHole_2.2mm_M2, F.Cu at (261.7, 88.9)
- added REF1: MountingHole_2.2mm_M2, MountingHole:MountingHole_2.2mm_M2, F.Cu at (261.7, 27.9)
- added REF2: MountingHole_2.2mm_M2, MountingHole:MountingHole_2.2mm_M2, F.Cu at (172.8, 27.9)
- added REF3: MountingHole_2.2mm_M2, MountingHole:MountingHole_2.2mm_M2, F.Cu at (172.8, 88.9)
- moved G*** 68.8 mm to (233.7, 68.6)
- moved J9 41.0 mm to (180.4, 81.3), turned to 0 degrees
- moved J10 36.6 mm to (188.0, 83.8), turned to 0 degrees
Connections:
- A1 pad 25: unconnected-(A1-Pad25) -> Net-(J11-Pad2)
Routing:
- net Net-(J11-Pad2): track 0.00 -> 32.4 mm
- net Net-(A1-Pad23): track 12.7 -> 38.0 mm
- net Net-(A1-Pad24): track 16.3 -> 37.8 mm
Other:
- board size 106.6 x 66 mm -> 93.9 x 66 mm
- board text added: "Servo Driver Interface Board v2.1 TALUS :: Autonomous Robotics Club 2022 Jim Moroney"
- board text removed: "Servo Driver Interface Board v1.0 TALUS :: Autonomous Robotics Club 2022 Jim Moroney"
