File: HARDWARE/ServoDriver/ArmDriver.kicad_sch (KiCad schematic)
At the start: 43 parts, among them J1 Conn_01x03_Male, J10 Screw_Terminal_01x02, J2 Conn_01x03_Male, J3 Conn_01x03_Male, J4 Conn_01x03_Male, J5 Conn_01x03_Male, J6 Conn_01x03_Male, J7 Conn_01x03_Male, J8 Conn_01x03_Male, J9 I2C Connector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

Commit message: ArmDriver rev2
Parts:
- added J11: Fan Connector, Connector_PinHeader_2.54mm:PinHeader_1x02_P2.54mm_Vertical, symbol Connector:Conn_01x02_Male
Connections:
- net GNDREF: now also J11.1 (Pin_1)
- net at A1.25 (A6): now also J11.2 (Pin_2)
Other:
- note added: "*A0-A3 pins used as surrogate digital pins"
- note removed: "*A0 & A1 pins used as surrogate digital pins"
Changed lines of the file:
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@@
+    (stroke (width 0) (type default) (color 0 0 0 0))
+  )
+  (wire (pts (xy 187.96 81.28) (xy 191.77 81.28))
     (stroke (width 0) (type default) (color 0 0 0 0))
   )
@@
     (effects (font (size 1.27 1.27)) (justify left bottom))
   )
-  (text "*A0 & A1 pins used as \n surrogate digital pins" (at 199.39 68.58 0)
+  (text "*A0-A3 pins used as \n surrogate digital pins" (at 199.39 68.58 0)
     (effects (font (size 1.27 1.27)) (justify left bottom))
   )
@@
     )
     (property "Datasheet" "" (id 3) (at 77.47 149.86 0)
+      (effects (font (size 1.27 1.27)) hide)
+    )
+    (pin "1")
+  )
+  (symbol (lib_id "power:GNDREF") (at 191.77 83.82 0) (unit 1)
+    (in_bom yes) (on_board yes)
+    (property "Reference" "#PWR0103" (id 0) (at 191.77 90.17 0)
+      (effects (font (size 1.27 1.27)) hide)
+    )
+    (property "Value" "GNDREF" (id 1) (at 191.897 88.2142 0))
+    (property "Footprint" "" (id 2) (at 191.77 83.82 0)
+      (effects (font (size 1.27 1.27)) hide)
+    )
+    (property "Datasheet" "" (id 3) (at 191.77 83.82 0)
       (effects (font (size 1.27 1.27)) hide)
     )
@@
     (pin "9")
   )
+  (symbol (lib_id "Connector:Conn_01x02_Male") (at 196.85 83.82 180) (unit 1)
+    (in_bom yes) (on_board yes) (fields_autoplaced)
+    (property "Reference" "J11" (id 0) (at 198.12 81.2799 0)
+      (effects (font (size 1.27 1.27)) (justify right))
+    )
+    (property "Value" "Fan Connector" (id 1) (at 198.12 83.8199 0)
+      (effects (font (size 1.27 1.27)) (justify right))
+    )
+    (property "Footprint" "Connector_PinHeader_2.54mm:PinHeader_1x02_P2.54mm_Vertical" (id 2) (at 196.85 83.82 0)
+      (effects (font (size 1.27 1.27)) hide)
+    )
+    (property "Datasheet" "~" (id 3) (at 196.85 83.82 0)
+      (effects (font (size 1.27 1.27)) hide)
+    )
+    (pin "1")
+    (pin "2")
+  )
   (symbol (lib_id "Connector:Screw_Terminal_01x02") (at 179.07 114.3 0) (mirror x) (unit 1)
     (in_bom yes) (on_board yes) (fields_autoplaced)
@@
       (reference "#PWR0102") (unit 1) (value "+5V") (footprint "")
     )
+    (path "/1e624c85-1e9d-4577-a218-3212aed0eda1"
+      (reference "#PWR0103") (unit 1) (value "GNDREF") (footprint "")
+    )
     (path "/d0e74642-b451-4818-8635-6c6460d97fb7"
       (reference "A1") (unit 1) (value "Arduino_Nano_v3.x") (footprint "Module:Arduino_Nano")
@@
       (reference "J10") (unit 1) (value "Screw_Terminal_01x02") (footprint "TerminalBlock:TerminalBlock_Altech_AK300-2_P5.00mm")
     )
+    (path "/d63769fb-fd44-487c-ac6d-09d1e60989cf"
+      (reference "J11") (unit 1) (value "Fan Connector") (footprint "Connector_PinHeader_2.54mm:PinHeader_1x02_P2.54mm_Vertical")
+    )
     (path "/00000000-0000-0000-0000-00005dcf6ff0"
